File: xiaomao.sch (KiCad schematic (older format))
At the start: 16 parts, among them J1 JTAG, J2 UART, J3 Conn_01x05, SW1 SW_Push, U1 SeeeduinoXIAO

Commit message: Add SW_SPST hole
Parts:
- SW1: footprint Button_Switch_SMD:SW_SPST_B3U-1000P -> Button_Switch_SMD:SW_SPST_B3U-1000P-B
Changed lines of the file:
@@
 encoding utf-8
 Sheet 1 1
-Title ""
-Date ""
-Rev ""
-Comp ""
+Title "Xiaomao"
+Date "2021-10-05"
+Rev "v0.2"
+Comp "Securing Hardware"
 Comment1 ""
 Comment2 ""
@@
 F 0 "SW1" V 5346 1652 50  0000 R CNN
 F 1 "SW_Push" V 5255 1652 50  0000 R CNN
-F 2 "Button_Switch_SMD:SW_SPST_B3U-1000P" H 5300 1900 50  0001 C CNN
+F 2 "Button_Switch_SMD:SW_SPST_B3U-1000P-B" H 5300 1900 50  0001 C CNN
 F 3 "~" H 5300 1900 50  0001 C CNN
 F 4 "C498294" H 5300 1700 50  0001 C CNN "LCSC"
